File: pcb files/4x3_derived.kicad_pcb (KiCad board)
At the start: 2 copper layers, 75 x 57.2 mm, 46 parts, among them J1 USB_C_Receptacle_USB2.0, J6 Conn_01x02_Socket, U1 STM32F072CBT6, U2 PRTR5V0U2X, U3 XC6206PxxxMR-Regulator_Linear

Commit message: pcb updated
Parts:
- added J5: Conn_01x02_Socket, Connector_PinHeader_2.54mm:PinHeader_1x02_P2.54mm_Vertical, F.Cu at (1.82, 1.82)
- added S13: Keyswitch, ScottoKeebs_Hotswap:Hotswap_MX_Plated_2.00u, F.Cu at (58.9, 84.5)
Routing:
- net col 2: track 27.7 -> 51.0 mm, vias 0 -> 2
- net col 0: track 74.8 -> 93.2 mm
- net Net-(D9-A): track 4.21 -> 18.2 mm
- net row 2: track 94.6 -> 97.8 mm, vias 2 -> 4
Other:
- board text added: "vtsoi 2026"
